File: hardware/kicad_session1/lri_s1/lri_s1.kicad_sch (KiCad schematic)
At the start: 49 parts, among them J1 USB_C_Receptacle_USB2.0_16P, J2 CTRL1, J3 CTRL2, J4 Micro_SD_Card, Q1 NMOS, SW1 MJTP1230, SW2 MJTP1230, U1 STM32F042F6P6, U2 LP5912-3.3DRV, U3 BMP390, U6 ICM-42688-P

Commit message: Simplified LED FET circuit, general BOM consolidation. First instance of layout, need to redo.
Parts:
- removed Q1: NMOS, symbol Simulation_SPICE:NMOS
- removed R7: 100, Resistor_SMD:R_0402_1005Metric, symbol Device:R_Small
- removed R8: 5.1k, Resistor_SMD:R_0201_0603Metric, symbol Device:R_Small
- removed SW1, SW2: MJTP1230, lib:MJTP1230, symbol Switch:SW_MEC_5E
- removed U6: ICM-42688-P, symbol lri_s1_symbols:ICM-42688-P
- added Q2: T2N7002AK, Package_TO_SOT_SMD:SOT-23, symbol Transistor_FET:T2N7002AK
- added SW1, SW2: SW_Push, Button_Switch_SMD:SW_SPST_PTS810, symbol Switch:SW_Push
- added U4: ICM-42688-P, lib:ICM-42688_LGA_0.91x2.50x3.00, symbol lri_s1_symbols:ICM-42688-P
- C1: footprint Capacitor_SMD:C_0603_1608Metric -> Capacitor_SMD:C_0402_1005Metric
- C16, C17: footprint (none) -> Capacitor_THT:CP_Radial_D5.0mm_P2.00mm
- C9: value 100n -> 10n
- F1, F2: footprint (none) -> Fuse:Fuse_0402_1005Metric
- J2, J3: footprint (none) -> Connector_PinSocket_2.54mm:PinSocket_1x03_P2.54mm_Vertical
- J4: footprint (none) -> Connector_Card:microSD_HC_Wuerth_693072010801
- R1, R12, R13: footprint Resistor_SMD:R_0201_0603Metric -> Resistor_SMD:R_0402_1005Metric
- U3: footprint (none) -> lib:BMP390_LGA_2x2x0.75
- renumbered R10 to R7, R11 to R8
Connections:
- net +3V3: now also SW1.1, SW2.2, U4.5 (VDDIO), U4.8 (VDD); no longer R1.1, U1.1 (PB8)
- net GND: now also R1.1, U1.1 (PB8), SW1.2, U4.10 (RESV), U4.11 (RESV), U4.2 (RESV), U4.3 (RESV), U4.6 (GND), U4.7 (RESV)
- net ICM_~{CS}: now also U4.12 (AP_CS)
- net LED: now also Q2.1 (G)
- net SPI1_MISO: now also U4.1 (A_SDO)
- net SPI1_MOSI: now also U4.14 (AP_SDI)
- net SPI1_SCK: now also U4.13 (AO_SCK)
- net at R1.2: now also SW2.1
- net at R6.1: now also Q2.3 (D)
- net at D2.2 (A): now also Q2.2 (S)

Commit message: Finished tutorial flight computer PCB, awaiting backcheck + merge.
Parts:
- removed C10: 10u, Capacitor_SMD:C_0402_1005Metric, symbol Device:C_Small
- renumbered C11 to C10, C12 to C11
Connections:
- net BMP_~{CS}: now also U1.9 (PA3); no longer U1.10 (PA4)
- net GPIO2: now also U1.8 (PA2); no longer U1.14 (PB1)
- net ICM_~{CS}: now also U1.14 (PB1); no longer U1.9 (PA3)
- net SD_~{CS}: now also U1.10 (PA4); no longer U1.8 (PA2)
- net SPI1_MOSI: now also U1.13 (PA7); no longer U1.11 (PA5)
- net SPI1_SCK: now also U1.11 (PA5); no longer U1.13 (PA7)
Other:
- moved on the sheet: C10, C11, U3

Commit message: Cleaned up layout
Parts:
- J4: footprint Connector_Card:microSD_HC_Wuerth_693072010801 -> Connector_Card:microSD_HC_Molex_47219-2001
Other:
- note added: "INERTIAL MEASUREMENT UNIT"
- note removed: "ACCELEROMETER + GYROSCOPE"
Changed lines of the file:
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@@
 		)
 	)
-	(text "ACCELEROMETER + GYROSCOPE"
+	(text "INERTIAL MEASUREMENT UNIT"
 		(exclude_from_sim no)
 		(at 177.8 154.686 0)
@@
 			)
 		)
-		(property "Footprint" "Connector_Card:microSD_HC_Wuerth_693072010801"
+		(property "Footprint" "Connector_Card:microSD_HC_Molex_47219-2001"
 			(at 148.59 151.13 0)
 			(effects
